Commit message: made wheel collision spheres to reduce friction with the floor, not sure if its working well enough. did not add xacro toggle between diffdrive and ros2control because it wasn't working and ros2 control will be used for the real robot anyways

File: dev_ws/src/dusty/description/robot_core.xacro (robot description, xacro)
@@ -45,5 +45,5 @@
     </link>
     <gazebo reference="chassis">
-        <material>Gazebo/White</material>
+        <material>Gazebo/Black</material>
     </gazebo>
     <!-- LEFT WHEEL LINK -->
@@ -63,5 +63,5 @@
         <collision>
             <geometry>
-                <cylinder radius="0.035" length="0.02"/>
+                <sphere radius="0.035"/>
             </geometry>
         </collision>
@@ -89,5 +89,5 @@
         <collision>
             <geometry>
-                <cylinder radius="0.035" length="0.02"/>
+                <sphere radius="0.035"/>
             </geometry>
         </collision>
